File: Chris Bidinosti/KVL+KCL/KVL+KCL.kicad_sch (KiCad schematic)
At the start: 10 parts

Commit message: Add files via upload
Parts:
- removed U1, U2, U3, U4, U5, U6: ~, banana_connector:Red&BlackBananaConnector, symbol banana_connector:red_and_black_banana_connectors
- added H1, H2, H3, H4, H5: MountingHole, MountingHole:MountingHole_3.2mm_M3, symbol Mechanical:MountingHole
- added J1, J2, J3, J4, J5: ~, jumper_connector:JumperConnector, symbol JumperConnector:banana_jumper
- added TP1, TP2, TP3, TP4: TestPoint, TestPoint:TestPoint_Pad_D2.5mm, symbol Connector:TestPoint
- added U1: ~, power_connector:power_connector, symbol PowerConnector:power_connector
Connections:
- net +1V5: now also TP1.1, U1.1 (V+)
- net GND: now also TP4.1, U1.2 (GND)
- net at R4.2: now also J5.2 (J-)
- net at R1.2: now also J1.1 (J+)
- net at R3.2: now also J3.2 (J-)
- net at R2.2, R3.1: now also J4.2 (J-), J5.1 (J+), TP3.1
- net at R2.1: now also J2.2 (J-)
- new net: J1.2 (J-), J2.1 (J+), J3.1 (J+), J4.1 (J+), TP2.1
