File: Russell Mammei/8thOrderBandpassFilter/8thOrderBandpassFilter.kicad_sch (KiCad schematic)
At the start: 36 parts, among them J1 Input, J2 Output, J3 Power, U1 ADA4177-2ARZ, U2 ADA4177-4ARZ-RL

Commit message: Add files via upload
Parts:
- C10, C12, C14, C16, C18, C3, C5, C7, C8, C9: Link (none) -> https://www.digikey.ca/en/products/detail/murata-electronic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
- C11, C13, C15, C17: Link (none) -> https://www.digikey.ca/en/products/detail/samsung-electro-m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
- C4, C6: Link (none) -> https://www.digikey.ca/en/products/detail/kemet/C0603C331F5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
- D1, D2: Link (none) -> https://www.digikey.ca/en/products/detail/littelfuse-inc/SM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
- D3: Link (none) -> https://www.digikey.ca/en/products/detail/yageo/SMAJ12CA-TR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
- J1: Link (none) -> https://www.digikey.ca/en/products/detail/amphenol-rf/031-5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
- R1, R10, R2, R3, R4, R5, R6, R7, R8, R9: Link (none) -> https://www.digikey.ca/en/products/detail/yageo/RT0603BRD07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
- U1, U2: Link (none) -> https://www.digikey.ca/en/products/detail/analog-devices-in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
