File: Russell Mammei/12VDualRailPowerSupply/12VDualRailPowerSupply.kicad_pcb (KiCad board)
At the start: 4 copper layers, 55 x 24 mm, 22 parts, among them J1 PJ-066A, U1 PDM2-S12-D15-S, U2 MC79L12ACDR, U3 AS78L12RTR-G1

Commit message: Add files via upload
Parts:
- C1, C2: value 4700nF -> 10uF
- L1: value 6800nH -> 5.6uH; footprint Inductor:IND_LQH3NPZ6R8MMEL -> SRN3015BTA:IND_SRN3015BTA-2R2M_BRN-L
- U1: value PDM2-S12-D15-S -> PCN2-S12-D15-S; footprint DCDCConverter:CONV_PDM2-S12-D15-S -> DCDCConverterNew:CONV_PCN2-S12-D15-S
- moved L1 0.10 mm to (135.6, 95.5), turned to 180 degrees
Connections:
- C2 pad 1: Net-(U1-VIN) -> Net-(U1-+VIN)
- L1 pad 1: /V_wall -> Net-(U1-+VIN)
- L1 pad 2: Net-(U1-VIN) -> /V_wall
- LED1 pad 1: GND -> Net-(LED1-Pad1)
- LED1 pad 2: Net-(LED1-Pad2) -> GND
- LED1 pad 3: Net-(LED1-Pad3) -> GND
- LED1 pad 4: GND -> Net-(LED1-Pad4)
- R1 pad 2: Net-(LED1-Pad3) -> Net-(LED1-Pad4)
- R2 pad 2: Net-(LED1-Pad2) -> Net-(LED1-Pad1)
- U1 pad 1: Net-(U1-VIN) -> Net-(U1-+VIN)
Routing:
- net Net-(LED1-Pad2): track 10.5 -> 0.00 mm
- net Net-(LED1-Pad3): track 8.79 -> 0.00 mm
- net Net-(LED1-Pad4): track 0.00 -> 6.71 mm
- net Net-(LED1-Pad1): track 0.00 -> 5.30 mm
- net Net-(U1-+VIN): track 0.00 -> 1.75 mm
- net Net-(U1-VIN): track 1.74 -> 0.00 mm
- added copper zone on B.Cu, net Net-(U1-+VIN)
- removed copper zone on B.Cu, net Net-(U1-VIN)
Other:
- board text added: "12V Dual Rail Power Supply V1.1. Tapendra BC, Aug 2026 Based On David Ostapchuck's Design"
- board text added: "C1/2 = 10uF C3/4 = 470nF C5/6 = 330nF C7/8 = 100nF"
- board text added: "L1 = 5600nH R1/2 = 1K FB1-3 = 2k @ 100MHZ"
- board text removed: "12V Dual Rail Power Supply V1.0. Tapendra BC, Aug 2026 Based On David Ostapchuck's Design"
- board text removed: "C1/2 = 4700nF C3/4 = 470nF C5/6 = 330nF C7/8 = 100nF"
- board text removed: "L1 = 6800nH R1/2 = 1K FB1-3 = 2k @ 100MHZ"
