File: Russell Mammei/12VDualRailPowerSupply/12VDualRailPowerSupply.kicad_sch (KiCad schematic)
At the start: 21 parts, among them J1 PJ-066A, U1 PDM2-S12-D15-S, U2 MC79L12ACDR, U3 AS78L12RTR-G1

Commit message: Add files via upload
Parts:
- removed L1: 6800nH, Inductor:IND_LQH3NPZ6R8MMEL, symbol Inductor:LQH3NPZ6R8MMEL
- removed U1: PDM2-S12-D15-S, DCDCConverter:CONV_PDM2-S12-D15-S, symbol DCDCConverter:PDM2-S12-D15-S
- added L1: 5.6uH, SRN3015BTA:IND_SRN3015BTA-2R2M_BRN-L, symbol SRN3015BTA:SRN3015BTA-5R6M
- added U1: PCN2-S12-D15-S, DCDCConverterNew:CONV_PCN2-S12-D15-S, symbol DCDCConverterNew:PCN2-S12-D15-S
- C1, C2: value 4700nF -> 10uF
- LED1: footprint IndicatorLED:SSF-LXHM250IGIGW_LUM -> SSF-LXHM250IGIGW_LUM
Connections:
- net GND: now also LED1.2, LED1.3, U1.5 (COMMON); no longer LED1.1, LED1.4
- net GND Wall: now also U1.2 (-VIN)
- net V+: now also U1.6 (+VOUT)
- net V-: now also U1.4 (-VOUT)
- net V_wall: now also L1.2
- net at R2.2: now also LED1.1; no longer LED1.2
- net at C2.1: now also L1.1, U1.1 (+VIN)
- net at R1.2: now also LED1.4; no longer LED1.3
Other:
- note added: "* PDM2 DC DC converter is discontinued, therefore it is replaced with PCN2 DC DC converter as per bel recommendation in V1.1"
- note added: "EMC Class B Filter"
